Commit message: fixed issue with tf and cmd_vel

File: src/bot_gazebo/urdf/bot.urdf.xacro (robot description, xacro)
@@ -34,73 +34,54 @@
     </collision>
   </link>
-  <!-- Left Wheel -->
-  <link name="left_wheel">
-    <inertial>
-      <origin xyz="0 0 0" rpy="0 0 0"/>
-      <mass value="${mass_wheel}"/>
-      <inertia ixx="0.01" ixy="0" ixz="0" iyy="0.01" iyz="0" izz="0.01"/>
-    </inertial>
-    <visual>
-      <origin xyz="0 0 0" rpy="${pi/2} 0 0"/>
-      <geometry>
-        <cylinder radius="${wheel_radius}" length="${wheel_width}"/>
-      </geometry>
-      <material name="wheel_color">
-        <color rgba="0.1 0.1 0.1 1.0"/>  <!-- Black -->
-      </material>
-    </visual>
-    <collision>
-      <origin xyz="0 0 0" rpy="${pi/2} 0 0"/>
-      <geometry>
-        <cylinder radius="${wheel_radius}" length="${wheel_width}"/>
-      </geometry>
-    </collision>
-  </link>
-  <!-- Right Wheel -->
-  <link name="right_wheel">
-    <inertial>
-      <origin xyz="0 0 0" rpy="0 0 0"/>
-      <mass value="${mass_wheel}"/>
-      <inertia ixx="0.01" ixy="0" ixz="0" iyy="0.01" iyz="0" izz="0.01"/>
-    </inertial>
-    <visual>
-      <origin xyz="0 0 0" rpy="${pi/2} 0 0"/>
-      <geometry>
-        <cylinder radius="${wheel_radius}" length="${wheel_width}"/>
-      </geometry>
-      <material name="wheel_color">
-        <color rgba="0.1 0.1 0.1 1.0"/>  <!-- Black -->
-      </material>
-    </visual>
-    <collision>
-      <origin xyz="0 0 0" rpy="${pi/2} 0 0"/>
-      <geometry>
-        <cylinder radius="${wheel_radius}" length="${wheel_width}"/>
-      </geometry>
-    </collision>
-  </link>
-  <!-- Caster Wheel (Front) -->
-  <link name="caster_wheel">
-    <inertial>
-      <origin xyz="0 0 0" rpy="0 0 0"/>
-      <mass value="0.3"/>
-      <inertia ixx="0.005" ixy="0" ixz="0" iyy="0.005" iyz="0" izz="0.005"/>
-    </inertial>
-    <visual>
-      <origin xyz="0 0 0" rpy="0 0 0"/>
-      <geometry>
-        <sphere radius="0.05"/>
-      </geometry>
-      <material name="wheel_color">
-        <color rgba="0.1 0.1 0.1 1.0"/>  <!-- Black -->
-      </material>
-    </visual>
-    <collision>
-      <origin xyz="0 0 0" rpy="0 0 0"/>
-      <geometry>
-        <sphere radius="0.05"/>
-      </geometry>
-    </collision>
-  </link>
+  <!-- Wheel macro, instantiated for all four corners below. Skid-steer
+       drivetrain; the left pair shares one Pololu G2 channel, the right
+       pair shares the other, so both wheels on a side always spin together
+       (matches the diff_drive plugin's multi-joint-per-side config below;
+       there is no caster, all four wheels are driven). -->
+  <xacro:macro name="wheel" params="prefix x_reflect y_reflect">
+    <link name="${prefix}_wheel">
+      <inertial>
+        <origin xyz="0 0 0" rpy="0 0 0"/>
+        <mass value="${mass_wheel}"/>
+        <inertia ixx="0.01" ixy="0" ixz="0" iyy="0.01" iyz="0" izz="0.01"/>
+      </inertial>
+      <visual>
+        <origin xyz="0 0 0" rpy="${pi/2} 0 0"/>
+        <geometry>
+          <cylinder radius="${wheel_radius}" length="${wheel_width}"/>
+        </geometry>
+        <material name="wheel_color">
+          <color rgba="0.1 0.1 0.1 1.0"/>  <!-- Black -->
+        </material>
+      </visual>
+      <collision>
+        <origin xyz="0 0 0" rpy="${pi/2} 0 0"/>
+        <geometry>
+          <cylinder radius="${wheel_radius}" length="${wheel_width}"/>
+        </geometry>
+      </collision>
+    </link>
+    <!-- type is "continuous" (not "revolute"). These are driven wheels and
+         need unlimited rotation. A revolute joint requires <limit> and a
+         lower=upper=0 limit (an earlier version of this file had exactly
+         that) welds the wheel at zero rotation, so it can never turn no
+         matter what the diff_drive plugin commands. -->
+    <joint name="${prefix}_wheel_joint" type="continuous">
+      <origin xyz="${x_reflect * wheelbase/2} ${y_reflect * track_width/2} ${wheel_radius}" rpy="0 0 0"/>
+      <parent link="base_link"/>
+      <child link="${prefix}_wheel"/>
+      <axis xyz="0 1 0"/>
+      <dynamics damping="0.1" friction="0.0"/>
+    </joint>
+    <gazebo reference="${prefix}_wheel">
+      <material>Gazebo/Black</material>
+      <mu1>0.8</mu1>
+      <mu2>0.8</mu2>
+    </gazebo>
+  </xacro:macro>
+  <xacro:wheel prefix="front_left" x_reflect="1" y_reflect="1"/>
+  <xacro:wheel prefix="rear_left" x_reflect="-1" y_reflect="1"/>
+  <xacro:wheel prefix="front_right" x_reflect="1" y_reflect="-1"/>
+  <xacro:wheel prefix="rear_right" x_reflect="-1" y_reflect="-1"/>
   <!-- Lidar Link -->
   <link name="lidar_link">
@@ -149,28 +130,4 @@
     </collision>
   </link>
-  <!-- Left Wheel Joint -->
-  <joint name="left_wheel_joint" type="revolute">
-    <origin xyz="0 ${track_width/2} ${wheel_radius}" rpy="0 0 0"/>
-    <parent link="base_link"/>
-    <child link="left_wheel"/>
-    <axis xyz="0 1 0"/>
-    <limit lower="0" upper="0" effort="30" velocity="1"/>
-    <dynamics damping="0.1" friction="0.0"/>
-  </joint>
-  <!-- Right Wheel Joint -->
-  <joint name="right_wheel_joint" type="revolute">
-    <origin xyz="0 ${-track_width/2} ${wheel_radius}" rpy="0 0 0"/>
-    <parent link="base_link"/>
-    <child link="right_wheel"/>
-    <axis xyz="0 1 0"/>
-    <limit lower="0" upper="0" effort="30" velocity="1"/>
-    <dynamics damping="0.1" friction="0.0"/>
-  </joint>
-  <!-- Caster Wheel Joint (Fixed to front center bottom) -->
-  <joint name="caster_wheel_joint" type="fixed">
-    <origin xyz="${base_length/2 - 0.08} 0 0.05" rpy="0 0 0"/>
-    <parent link="base_link"/>
-    <child link="caster_wheel"/>
-  </joint>
   <!-- Lidar Joint -->
   <joint name="lidar_joint" type="fixed">
@@ -189,24 +146,16 @@
     <material>Gazebo/Blue</material>
   </gazebo>
-  <gazebo reference="left_wheel">
-    <material>Gazebo/Black</material>
-    <mu1>0.8</mu1>
-    <mu2>0.8</mu2>
-  </gazebo>
-  <gazebo reference="right_wheel">
-    <material>Gazebo/Black</material>
-    <mu1>0.8</mu1>
-    <mu2>0.8</mu2>
-  </gazebo>
-  <gazebo reference="caster_wheel">
-    <material>Gazebo/Gray</material>
-    <mu1>0.3</mu1>
-    <mu2>0.3</mu2>
-  </gazebo>
-  <!-- Differential Drive Plugin (gz-sim) -->
+  <!-- Differential (skid-steer) Drive Plugin (gz-sim). Two joints per side,
+       matching the real drivetrain; the Pololu G2's left channel drives
+       front_left+rear_left together, right channel drives
+       front_right+rear_right together, and this plugin commands both
+       joints on a side identically, same as the real motor driver does
+       electrically. -->
   <gazebo>
     <plugin filename="gz-sim-diff-drive-system" name="gz::sim::systems::DiffDrive">
-      <left_joint>left_wheel_joint</left_joint>
-      <right_joint>right_wheel_joint</right_joint>
+      <left_joint>front_left_wheel_joint</left_joint>
+      <left_joint>rear_left_wheel_joint</left_joint>
+      <right_joint>front_right_wheel_joint</right_joint>
+      <right_joint>rear_right_wheel_joint</right_joint>
       <wheel_separation>${track_width}</wheel_separation>
       <wheel_radius>${wheel_radius}</wheel_radius>
@@ -219,4 +168,9 @@
       <odom_publish_frequency>30</odom_publish_frequency>
     </plugin>
+    <!-- Publishes joint positions on gz-transport so robot_state_publisher
+         can compute base_link -> *_wheel TF. Without this the wheel joints
+         are non-fixed (continuous) but nothing reports their position, so
+         robot_state_publisher has nothing to publish their transform from. -->
+    <plugin filename="gz-sim-joint-state-publisher-system" name="gz::sim::systems::JointStatePublisher"/>
   </gazebo>
   <!-- Lidar Sensor (simulates RPLIDAR) - gz-sim gpu_lidar -->

Commit message: did whatever

File: src/bot_gazebo/urdf/bot.urdf.xacro (robot description, xacro)
@@ -145,4 +145,22 @@
   <gazebo reference="base_link">
     <material>Gazebo/Blue</material>
+    <!-- Diagnostic contact sensor - publishes actual collision events for
+         base_link so real collisions (e.g. clipping a bale) can be observed
+         directly instead of inferred from TF/cmd_vel mismatches. Requires
+         the gz-sim-contact-system plugin to be loaded on the world (see
+         bot_gazebo/worlds/*_cfr.world) - unlike camera/lidar, contact
+         sensors produce no output at all without it. "collision" is
+         sdformat_urdf's default generated name for base_link's single,
+         unnamed URDF <collision> element; if this sensor stays silent,
+         verify the real name via `gz topic -l | grep contact`.
+         An explicit <topic> avoids having to guess gz-sim's auto-generated
+         hierarchical topic name when bridging in gazebo_sim.launch.py. -->
+    <sensor name="base_contact_sensor" type="contact">
+      <contact>
+        <collision>collision</collision>
+        <topic>/bot_contacts</topic>
+      </contact>
+      <update_rate>30</update_rate>
+    </sensor>
   </gazebo>
   <!-- Differential (skid-steer) Drive Plugin (gz-sim). Two joints per side,

Commit message: updated bot dimensions, fixed issues with planner. Bot is mapping now but slow

File: src/bot_gazebo/urdf/bot.urdf.xacro (robot description, xacro)
@@ -2,13 +2,13 @@
 <robot xmlns:xacro="http://www.ros.org/wiki/xacro" name="bot">
   <!-- Constants -->
-  <xacro:property name="base_length" value="0.61"/>  <!-- 24 inches -->
-  <xacro:property name="base_width" value="0.41"/>   <!-- 16 inches -->
-  <xacro:property name="base_height" value="0.15"/>  <!-- chassis height -->
-  <xacro:property name="wheel_radius" value="0.1"/>  <!-- wheel radius -->
-  <xacro:property name="wheel_width" value="0.08"/>  <!-- wheel width -->
-  <xacro:property name="wheelbase" value="0.50"/>    <!-- distance between wheels -->
-  <xacro:property name="track_width" value="0.35"/>  <!-- width between wheel centers -->
-  <xacro:property name="mass_base" value="11.3"/>    <!-- 25 lbs in kg -->
-  <xacro:property name="mass_wheel" value="0.5"/>
+  <xacro:property name="base_length" value="0.45"/>  <!-- 17.7 inches -->
+  <xacro:property name="base_width" value="0.27"/>   <!-- 10.6inches -->
+  <xacro:property name="base_height" value="0.176"/>  <!-- chassis height -->
+  <xacro:property name="wheel_radius" value="0.12"/>  <!-- wheel radius -->
+  <xacro:property name="wheel_width" value="0.06"/>  <!-- wheel width -->
+  <xacro:property name="wheelbase" value="0.33"/>    <!-- distance between wheels -->
+  <xacro:property name="track_width" value="0.22"/>  <!-- width between wheel centers -->
+  <xacro:property name="mass_base" value="3.2"/>    <!-- 7 lbs  -->
+  <xacro:property name="mass_wheel" value="0.2"/>
   <!-- Base Link (Chassis) -->
   <link name="base_link">

Commit message: Added new planning config and test script for nav2

File: src/bot_gazebo/urdf/bot.urdf.xacro (robot description, xacro)
@@ -130,4 +130,27 @@
     </collision>
   </link>
+  <!-- IMU Link -->
+  <link name="imu_link">
+    <inertial>
+      <origin xyz="0 0 0" rpy="0 0 0"/>
+      <mass value="0.05"/>
+      <inertia ixx="0.00001" ixy="0" ixz="0" iyy="0.00001" iyz="0" izz="0.00001"/>
+    </inertial>
+    <visual>
+      <origin xyz="0 0 0" rpy="0 0 0"/>
+      <geometry>
+        <box size="0.02 0.02 0.01"/>
+      </geometry>
+      <material name="imu_color">
+        <color rgba="0.9 0.1 0.1 1.0"/>  <!-- Red -->
+      </material>
+    </visual>
+    <collision>
+      <origin xyz="0 0 0" rpy="0 0 0"/>
+      <geometry>
+        <box size="0.02 0.02 0.01"/>
+      </geometry>
+    </collision>
+  </link>
   <!-- Lidar Joint -->
   <joint name="lidar_joint" type="fixed">
@@ -141,4 +164,13 @@
     <parent link="base_link"/>
     <child link="camera_link"/>
+  </joint>
+  <!-- IMU Joint, mounted flush at the chassis center (no offset needed
+       the way lidar/camera need clearance/forward placement), x-forward
+       z-up matching base_link's own axes so imu_link's orientation
+       readings need no extra rotation to interpret in base_link/odom. -->
+  <joint name="imu_joint" type="fixed">
+    <origin xyz="0 0 ${base_height/2}" rpy="0 0 0"/>
+    <parent link="base_link"/>
+    <child link="imu_link"/>
   </joint>
   <!-- Gazebo plugins -->
@@ -162,4 +194,40 @@
       </contact>
       <update_rate>30</update_rate>
+    </sensor>
+  </gazebo>
+  <!-- IMU sensor (real part: Bosch BNO055) - feeds robot_localization's EKF
+       (see bot_bringup/config/ekf_params.yaml) so heading is tracked from
+       gyro/orientation between SLAM scan-match corrections, not just wheel
+       odometry. Requires the gz-sim-imu-system plugin loaded on the world
+       (see bot_gazebo/worlds/*_cfr.world) - same story as the contact
+       sensor above, it produces no output at all without it.
+       Noise stddevs below are approximated from the BNO055 datasheet's
+       noise-density specs (gyro ~0.014 deg/s/sqrt(Hz), accel ~150
+       ug/sqrt(Hz)), converted to a per-sample stddev at this sensor's
+       100Hz update_rate via stddev = density * sqrt(update_rate/2). This
+       is a standard approximation (treats the sensor as white noise
+       band-limited to Nyquist), not a substitute for validating against
+       the actual datasheet or real-hardware calibration once the BNO055
+       is mounted - see CLAUDE.md's open items. gz-sim's IMU sensor has no
+       way to attach noise/covariance to the orientation output itself
+       (only angular_velocity/linear_acceleration below); its
+       orientation_covariance will read back all-zero regardless. -->
+  <gazebo reference="imu_link">
+    <sensor name="imu_sensor" type="imu">
+      <always_on>true</always_on>
+      <update_rate>100</update_rate>
+      <topic>/imu</topic>
+      <imu>
+        <angular_velocity>
+          <x><noise type="gaussian"><mean>0.0</mean><stddev>0.0017</stddev></noise></x>
+          <y><noise type="gaussian"><mean>0.0</mean><stddev>0.0017</stddev></noise></y>
+          <z><noise type="gaussian"><mean>0.0</mean><stddev>0.0017</stddev></noise></z>
+        </angular_velocity>
+        <linear_acceleration>
+          <x><noise type="gaussian"><mean>0.0</mean><stddev>0.0104</stddev></noise></x>
+          <y><noise type="gaussian"><mean>0.0</mean><stddev>0.0104</stddev></noise></y>
+          <z><noise type="gaussian"><mean>0.0</mean><stddev>0.0104</stddev></noise></z>
+        </linear_acceleration>
+      </imu>
     </sensor>
   </gazebo>

Commit message: Fix sim heading/costmap/localization issues found during nav2 testing
- bot.urdf.xacro: name base_link's collision so the contact sensor
  actually matches it (was silently dead against the wrong auto-generated
  name); pin JointStatePublisher to a fixed 'joint_states' topic instead
  of the world-namespaced default; raise lidar mount height for wheel
  clearance margin
- gazebo_sim.launch.py: default world switched to speed_course_cfr;
  bridge the fixed joint_states topic
- speed_course_cfr.world, obstacle_course_cfr.world: split the
  start-signal gantry's solid-slab collision into two side posts so the
  gate is actually open (was blocking the start and phantom-walling the
  costmap)
- nav2_params*.yaml (4 files): lower inflation_radius 0.55->0.35 to clear
  the slalom lane centerline; add OAK-D voxel_layer to the global
  costmap; fix stale/wrong amcl initial_pose to match speed_course_cfr's
  real spawn; correct behavior_server config (was using ignored pre-Jazzy
  recovery_server keys, silently running default behaviors instead of the
  intended spin/backup/drive_on_heading/wait set)
- nav2_mapping_params*.yaml (4 files): same behavior_server fix; add
  OAK-D voxel_layer to the global costmap
- mapping.launch.py: supporting launch wiring for the above
- third_party/: removed, unused
- docker/README.md: add (previously untracked)
- docker/Dockerfile: rename from DockerFile

File: src/bot_gazebo/urdf/bot.urdf.xacro (robot description, xacro)
@@ -27,5 +27,5 @@
       </material>
     </visual>
-    <collision>
+    <collision name="base_collision">
       <origin xyz="0 0 ${base_height/2}" rpy="0 0 0"/>
       <geometry>
@@ -155,5 +155,7 @@
   <!-- Lidar Joint -->
   <joint name="lidar_joint" type="fixed">
-    <origin xyz="0 0 ${base_height + 0.06}" rpy="0 0 0"/>
+    <!-- +0.12 (was +0.06): puts the scan plane at ~0.296m, clear of the
+         wheel tops (~0.24m) so the lidar can't graze its own wheels. -->
+    <origin xyz="0 0 ${base_height + 0.12}" rpy="0 0 0"/>
     <parent link="base_link"/>
     <child link="lidar_link"/>
@@ -182,13 +184,14 @@
          the gz-sim-contact-system plugin to be loaded on the world (see
          bot_gazebo/worlds/*_cfr.world) - unlike camera/lidar, contact
-         sensors produce no output at all without it. "collision" is
-         sdformat_urdf's default generated name for base_link's single,
-         unnamed URDF <collision> element; if this sensor stays silent,
-         verify the real name via `gz topic -l | grep contact`.
+         sensors produce no output at all without it. The referenced
+         collision name must match base_link's <collision name="...">
+         above: sdformat_urdf does NOT name an unnamed URDF collision
+         "collision" (it uses <link>_collision), so the name is set
+         explicitly on both sides to avoid a silent no-match.
          An explicit <topic> avoids having to guess gz-sim's auto-generated
          hierarchical topic name when bridging in gazebo_sim.launch.py. -->
     <sensor name="base_contact_sensor" type="contact">
       <contact>
-        <collision>collision</collision>
+        <collision>base_collision</collision>
         <topic>/bot_contacts</topic>
       </contact>
@@ -257,6 +260,13 @@
          can compute base_link -> *_wheel TF. Without this the wheel joints
          are non-fixed (continuous) but nothing reports their position, so
-         robot_state_publisher has nothing to publish their transform from. -->
-    <plugin filename="gz-sim-joint-state-publisher-system" name="gz::sim::systems::JointStatePublisher"/>
+         robot_state_publisher has nothing to publish their transform from.
+         Explicit <topic> pins a fixed name instead of the default
+         /world/<world>/model/<model>/joint_state, whose <world> segment is
+         the world file's INTERNAL name (e.g. cfr_speed_course), not its
+         filename/launch-arg (speed_course_cfr), bridging the auto name
+         would silently miss, leaving no wheel links in TF. -->
+    <plugin filename="gz-sim-joint-state-publisher-system" name="gz::sim::systems::JointStatePublisher">
+      <topic>joint_states</topic>
+    </plugin>
     <!-- Ground-truth pose publisher, sim-only diagnostic, NOT part of the
          real robot's sensor suite. DiffDrive's /odom above is kinematic

Commit message: fixed issue with bot not rotating, new issue with numpy error

File: src/bot_gazebo/urdf/bot.urdf.xacro (robot description, xacro)
@@ -5,4 +5,10 @@
   <xacro:property name="base_width" value="0.27"/>   <!-- 10.6inches -->
   <xacro:property name="base_height" value="0.176"/>  <!-- chassis height -->
+  <!-- Gap between the ground and the underside of the chassis. Without it
+       the chassis box was modelled spanning z=0..base_height, i.e. sitting
+       flat on the floor rather than riding on the wheels. That is wrong on
+       its own terms, though it was not what blocked turning: see the wheel
+       friction block below for that. -->
+  <xacro:property name="ground_clearance" value="0.06"/>
   <xacro:property name="wheel_radius" value="0.12"/>  <!-- wheel radius -->
   <xacro:property name="wheel_width" value="0.06"/>  <!-- wheel width -->
@@ -19,5 +25,5 @@
     </inertial>
     <visual>
-      <origin xyz="0 0 ${base_height/2}" rpy="0 0 0"/>
+      <origin xyz="0 0 ${ground_clearance + base_height/2}" rpy="0 0 0"/>
       <geometry>
         <box size="${base_length} ${base_width} ${base_height}"/>
@@ -28,5 +34,5 @@
     </visual>
     <collision name="base_collision">
-      <origin xyz="0 0 ${base_height/2}" rpy="0 0 0"/>
+      <origin xyz="0 0 ${ground_clearance + base_height/2}" rpy="0 0 0"/>
       <geometry>
         <box size="${base_length} ${base_width} ${base_height}"/>
@@ -76,6 +82,32 @@
     <gazebo reference="${prefix}_wheel">
       <material>Gazebo/Black</material>
-      <mu1>0.8</mu1>
-      <mu2>0.8</mu2>
+      <!-- Anisotropic tyre friction. This is what makes skid-steer
+           pivoting possible at all: a 4-wheel skid-steer can only rotate
+           by scrubbing all four tyres sideways, so lateral friction (mu1,
+           along fdir1) is low while rolling traction (mu2) stays high.
+           fdir1 is the WHEEL AXLE direction, but written as "0 0 1"
+           because fdir1 is expressed in the COLLISION frame and the
+           collision above is rotated rpy="pi/2 0 0", which maps the link's
+           Y axis onto the collision's Z. Getting this wrong is not a
+           subtle inaccuracy, it silently disables the whole friction
+           split: "0 1 0" here points along the contact normal, which is
+           degenerate, so the engine discards it and picks an arbitrary
+           direction. With that (and with the earlier isotropic 0.8/0.8)
+           the robot could not rotate AT ALL: a commanded 1.0 rad/s gave
+           exactly 0 deg of yaw while the wheels counter-rotated correctly,
+           so wheel odometry integrated turns that never happened and
+           heading was lost at every turn. With fdir1 correct, a 10s pivot
+           at 1.0 rad/s yields ~443 deg of real rotation.
+           The axle is also the only spin-invariant axis to aim fdir1
+           along: the wheel link rotates about it, so the friction split
+           stays put instead of tumbling with the wheel.
+           No <slip1>/<slip2> are set. They are not needed here: the
+           anisotropy alone reproduces realistic scrub (wheel odometry
+           over-reports a pivot by ~28%, which is why ekf_params.yaml gives
+           yaw to the IMU rather than the wheels). Add slip compliance only
+           if tyre modelling needs to get finer. -->
+      <mu1>0.05</mu1>
+      <mu2>1.0</mu2>
+      <fdir1>0 0 1</fdir1>
     </gazebo>
   </xacro:macro>
@@ -218,4 +250,13 @@
   <gazebo reference="imu_link">
     <sensor name="imu_sensor" type="imu">
+      <!-- Same reason as the lidar/camera sensors: without this the
+           bridged message carries gz's scoped sensor name
+           ("bot/base_link/imu_sensor") as its frame_id. That frame is not
+           in the TF tree, so robot_localization cannot transform the IMU
+           into base_link and silently DROPS every sample: the EKF's yaw
+           then sat at 0 while the IMU itself was correctly reporting the
+           turn, which is the whole reason imu0 exists in
+           ekf_params.yaml. -->
+      <gz_frame_id>imu_link</gz_frame_id>
       <always_on>true</always_on>
       <update_rate>100</update_rate>
