Commit message: Bring up real sensors on the Pi 5 and make launches robust on hardware
Lidar: the unit is an RPLIDAR S2 (1 Mbaud, DenseBoost). The apt
rplidar_ros driver segfaults on it, so hardware.launch.py now runs
Slamtec's sllidar_ros2 (built from source, gitignored, fetched at a
pinned commit by setup_pi.sh) with rplidar_params.yaml.

IMU: I2C1 on GPIO2/3 times out on this Pi even with nothing attached, so
the BNO055 moved to I2C3 on GPIO22/23 (pins 15/16). hardware.launch.py
takes an imu_i2c_bus arg (default 3); setup_pi.sh adds the
i2c3-pi5,pins_22_23 overlay; check_hardware.sh checks bus 3.

Launch fixes:
- Scope the OAK-D include in a GroupAction: depthai's camera.launch.py
  leaked use_composition='true' into nav2_bringup, which then died with
  "name 'true' is not defined".
- Skip RViz with a log line when rviz2 isn't installed instead of
  crashing midway and orphaning nodes that keep holding the lidar port
  and motor GPIO.
- Add sensor_view.launch.py + sensors.rviz: hardware layer + RViz
  anchored at base_link, for checking sensors without odom or a map.

Cleanup: split into clean_robot.sh (stops workspace nodes and anything
holding a sensor device via fuser, SIGINT first so motor_node shuts the
driver down, then drives the motor pins low) and clean_sim.sh (general
ROS/Gazebo cleanup, which clean_robot.sh calls).

URDF: place the OAK-D and lidar from measurements on the robot (OAK
front panel at the front edge, bottom 9 cm up; lidar 3.5 cm behind it,
0.95 cm right of its centre, top 5 cm above its top) and use the real
S2 and OAK-D S2 housing sizes.

Docs: README gets Pi setup, preflight, device table and troubleshooting,
and drops stale pigpio / rplidar_ros / sensor_fusion / goal_x content;
CLAUDE.md records the hardware findings and resolves a committed merge
conflict.

Co-Authored-By: Claude Opus 5.5 <noreply@anthropic.com>

File: src/bot_gazebo/urdf/bot.urdf.xacro (robot description, xacro)
@@ -17,4 +17,28 @@
   <xacro:property name="mass_base" value="3.2"/>    <!-- 3.2 kg = 7.0 lb -->
   <xacro:property name="mass_wheel" value="0.2"/>   <!-- 0.2 kg = 0.44 lb each -->
+  <!-- OAK-D S2 housing (~91 x 28 x 17.5 mm) and its measured mount height:
+       bottom of the housing 9 cm above the ground (measured 2026-09-25).
+       camera_link is the housing centre, which is also where
+       depthai_ros_driver hangs its oak-* optical frames (parent_frame). -->
+  <xacro:property name="oak_width" value="0.091"/>
+  <xacro:property name="oak_height" value="0.028"/>
+  <xacro:property name="oak_depth" value="0.0175"/>
+  <xacro:property name="oak_bottom_height" value="0.09"/>
+  <!-- Sensor placement, measured on the robot 2026-09-25 (relative to the
+       OAK housing, which is easy to measure against):
+       - OAK front panel is the robot's front edge (its 3 cm stand-off from
+         the chassis is already inside base_length), on the centreline
+         (lateral position assumed, not measured).
+       - Lidar centre is 3.5 cm behind the OAK front panel, 5.5 cm from the
+         OAK's left edge (i.e. 0.95 cm right of the OAK centre), and the
+         lidar top is 5 cm above the OAK top.
+       RPLIDAR S2 body is 77 mm dia x 38.85 mm tall (datasheet). lidar_link
+       sits on the scan plane, estimated 13 mm below the top of the head
+       (not measured; check against the window slit on the rotating head). -->
+  <xacro:property name="oak_front_x" value="${base_length/2}"/>
+  <xacro:property name="lidar_radius" value="0.0385"/>
+  <xacro:property name="lidar_body_height" value="0.03885"/>
+  <xacro:property name="lidar_top_height" value="${oak_bottom_height + oak_height + 0.05}"/>
+  <xacro:property name="lidar_plane_below_top" value="0.013"/>
   <!-- Base Link (Chassis) -->
   <link name="base_link">
@@ -124,7 +148,7 @@
     </inertial>
     <visual>
-      <origin xyz="0 0 0" rpy="0 0 0"/>
-      <geometry>
-        <cylinder radius="0.04" length="0.08"/>
+      <origin xyz="0 0 ${lidar_plane_below_top - lidar_body_height/2}" rpy="0 0 0"/>
+      <geometry>
+        <cylinder radius="${lidar_radius}" length="${lidar_body_height}"/>
       </geometry>
       <material name="lidar_color">
@@ -133,7 +157,7 @@
     </visual>
     <collision>
-      <origin xyz="0 0 0" rpy="0 0 0"/>
-      <geometry>
-        <cylinder radius="0.04" length="0.08"/>
+      <origin xyz="0 0 ${lidar_plane_below_top - lidar_body_height/2}" rpy="0 0 0"/>
+      <geometry>
+        <cylinder radius="${lidar_radius}" length="${lidar_body_height}"/>
       </geometry>
     </collision>
@@ -149,5 +173,5 @@
       <origin xyz="0 0 0" rpy="0 0 0"/>
       <geometry>
-        <box size="0.08 0.12 0.06"/>
+        <box size="${oak_depth} ${oak_width} ${oak_height}"/>
       </geometry>
       <material name="camera_color">
@@ -158,5 +182,5 @@
       <origin xyz="0 0 0" rpy="0 0 0"/>
       <geometry>
-        <box size="0.08 0.12 0.06"/>
+        <box size="${oak_depth} ${oak_width} ${oak_height}"/>
       </geometry>
     </collision>
@@ -185,20 +209,21 @@
     </collision>
   </link>
-  <!-- Lidar Joint -->
+  <!-- Lidar Joint. base_link's origin is at ground level (wheels are
+       centred at z=wheel_radius, so they touch the floor), so z IS the scan
+       plane's height above ground: ~0.155 m, above the OAK's top (0.118 m)
+       so the beam clears the camera. Measured position: see the sensor
+       placement properties at the top of this file. The live scan confirms
+       no self-returns (nothing closer than 0.32 m, 2026-09-25). -->
   <joint name="lidar_joint" type="fixed">
-    <!-- 0.1143m = 4.5in above the ground, matching the RPLIDAR's planned
-         mount height on the real robot. base_link's origin is at ground
-         level (wheels are radius 0.12 centred at z=0.12, so they touch the
-         floor), so this z IS the height above ground directly. Mounting
-         this low is safe despite the 360-degree scan: the wheels (~0.11m
-         out) and chassis body are both inside the sensor's 0.3m
-         <range><min> dead zone, so they never produce self-returns. -->
-    <origin xyz="0 0 0.1143" rpy="0 0 0"/>
+    <origin xyz="${oak_front_x - 0.035} ${oak_width/2 - 0.055} ${lidar_top_height - lidar_plane_below_top}" rpy="0 0 0"/>
     <parent link="base_link"/>
     <child link="lidar_link"/>
   </joint>
-  <!-- Camera Joint -->
+  <!-- Camera Joint. z is measured (base_link's origin is at ground level,
+       see lidar_joint): housing bottom at oak_bottom_height, so its centre
+       is half a housing-height above that (~0.104 m), below the lidar's
+       scan plane. x puts the front panel at the robot's front edge. -->
   <joint name="camera_joint" type="fixed">
-    <origin xyz="${base_length/2 - 0.05} 0 ${base_height/2 + 0.05}" rpy="0 0 0"/>
+    <origin xyz="${oak_front_x - oak_depth/2} 0 ${oak_bottom_height + oak_height/2}" rpy="0 0 0"/>
     <parent link="base_link"/>
     <child link="camera_link"/>

Commit message: Set the IMU's measured mount position and orientation in the URDF
Mounted 11.5 cm behind the chassis front panel, on the centreline,
94 mm up, with its X axis facing backwards (Y right, Z up), so imu_joint
is yaw = pi. bno055_node does no axis remapping, so with yaw 0 the EKF's
fused heading came out 180 deg off. Adds chassis_front_x (3 cm behind
the OAK face) so panel-relative measurements have a named reference.

Co-Authored-By: Claude Opus 5.5 <noreply@anthropic.com>

File: src/bot_gazebo/urdf/bot.urdf.xacro (robot description, xacro)
@@ -37,4 +37,8 @@
        (not measured; check against the window slit on the rotating head). -->
   <xacro:property name="oak_front_x" value="${base_length/2}"/>
+  <!-- The chassis front panel itself, 3 cm behind the OAK's front face
+       (the OAK stands proud of the panel, see above). Measure mount
+       positions "from the front panel" against this, not base_length/2. -->
+  <xacro:property name="chassis_front_x" value="${oak_front_x - 0.03}"/>
   <xacro:property name="lidar_radius" value="0.0385"/>
   <xacro:property name="lidar_body_height" value="0.03885"/>
@@ -229,10 +233,15 @@
     <child link="camera_link"/>
   </joint>
-  <!-- IMU Joint, mounted flush at the chassis center (no offset needed
-       the way lidar/camera need clearance/forward placement), x-forward
-       z-up matching base_link's own axes so imu_link's orientation
-       readings need no extra rotation to interpret in base_link/odom. -->
+  <!-- IMU Joint, measured on the robot 2026-09-28: 11.5 cm back from
+       the chassis front panel (not counting the OAK), 12.5 cm in from the
+       chassis left side (not counting the tyres), 94 mm above ground.
+       Mounted with its X axis facing the BACK of the robot, Y right, Z up:
+       base_link turned 180 deg about Z, hence yaw = pi. bno055_node does
+       no axis remapping of its own, so this transform is the only thing
+       that turns the chip's readings into base_link's frame for
+       robot_localization. With yaw 0 here, the fused absolute heading
+       comes out 180 deg off. -->
   <joint name="imu_joint" type="fixed">
-    <origin xyz="0 0 ${base_height/2}" rpy="0 0 0"/>
+    <origin xyz="${chassis_front_x - 0.115} ${base_width/2 - 0.125} 0.094" rpy="0 0 ${pi}"/>
     <parent link="base_link"/>
     <child link="imu_link"/>

Commit message: URDF: measured wheelbase 0.216 m (was a 0.33 estimate)
Co-Authored-By: Claude Opus 5.5 <noreply@anthropic.com>

File: src/bot_gazebo/urdf/bot.urdf.xacro (robot description, xacro)
@@ -13,5 +13,5 @@
   <xacro:property name="wheel_radius" value="0.06"/>  <!-- 0.06 m = 2.4 in radius (4.7 in dia) -->
   <xacro:property name="wheel_width" value="0.06"/>  <!-- 0.06 m = 2.4 in -->
-  <xacro:property name="wheelbase" value="0.33"/>    <!-- front-to-rear axle spacing, 0.33 m = 13.0 in -->
+  <xacro:property name="wheelbase" value="0.216"/>   <!-- front-to-rear axle spacing, measured 0.216 m = 8.5 in (2026-09-30; was a 0.33 estimate) -->
   <xacro:property name="track_width" value="0.32"/>  <!-- left-to-right wheel-centre spacing, 0.32 m = 12.6 in -->
   <xacro:property name="mass_base" value="3.2"/>    <!-- 3.2 kg = 7.0 lb -->

Commit message: Measured track width 0.33 m (was 0.32); fix two stale odometry tests
- URDF track_width, motor_node/wheel_odom_node track_width_m, drive_lib
- Nav2 footprint half-width 0.19 -> 0.195 in all 9 params files
- wheel_odom tests sent ticks_per_rev (979.62) as the encoder count; the
  node correctly rejects fractional counts, so they had failed since the
  real CPR went in on 09-24. Now whole counts, plus a test that fractional
  lines are ignored.

Co-Authored-By: Claude Opus 5.5 <noreply@anthropic.com>

File: src/bot_gazebo/urdf/bot.urdf.xacro (robot description, xacro)
@@ -14,5 +14,5 @@
   <xacro:property name="wheel_width" value="0.06"/>  <!-- 0.06 m = 2.4 in -->
   <xacro:property name="wheelbase" value="0.216"/>   <!-- front-to-rear axle spacing, measured 0.216 m = 8.5 in (2026-09-30; was a 0.33 estimate) -->
-  <xacro:property name="track_width" value="0.32"/>  <!-- left-to-right wheel-centre spacing, 0.32 m = 12.6 in -->
+  <xacro:property name="track_width" value="0.33"/>  <!-- left-to-right wheel-centre spacing, measured 0.33 m = 13.0 in (2026-09-30; was 0.32) -->
   <xacro:property name="mass_base" value="3.2"/>    <!-- 3.2 kg = 7.0 lb -->
   <xacro:property name="mass_wheel" value="0.2"/>   <!-- 0.2 kg = 0.44 lb each -->

Commit message: URDF: measured base mass 3.546 kg; box inertia from the dimensions
Inertia was a hardcoded 0.3/0.5/0.3 kg m^2 (~5-10x too high for a
3.5 kg 0.45x0.39 m box); now computed from mass_base and base_*.

Co-Authored-By: Claude Opus 5.5 <noreply@anthropic.com>

File: src/bot_gazebo/urdf/bot.urdf.xacro (robot description, xacro)
@@ -15,5 +15,5 @@
   <xacro:property name="wheelbase" value="0.216"/>   <!-- front-to-rear axle spacing, measured 0.216 m = 8.5 in (2026-09-30; was a 0.33 estimate) -->
   <xacro:property name="track_width" value="0.33"/>  <!-- left-to-right wheel-centre spacing, measured 0.33 m = 13.0 in (2026-09-30; was 0.32) -->
-  <xacro:property name="mass_base" value="3.2"/>    <!-- 3.2 kg = 7.0 lb -->
+  <xacro:property name="mass_base" value="3.545729"/>  <!-- measured 3.546 kg = 7.8 lb (2026-09-30; was 3.2) -->
   <xacro:property name="mass_wheel" value="0.2"/>   <!-- 0.2 kg = 0.44 lb each -->
   <!-- OAK-D S2 housing (~91 x 28 x 17.5 mm) and its measured mount height:
@@ -50,5 +50,11 @@
       <origin xyz="0 0 0" rpy="0 0 0"/>
       <mass value="${mass_base}"/>
-      <inertia ixx="0.3" ixy="0" ixz="0" iyy="0.5" iyz="0" izz="0.3"/>
+      <!-- Solid-box inertia from the mass and chassis dimensions (was a
+           hardcoded 0.3/0.5/0.3, 4-13x too large for a 3.5 kg box, which made
+           simulated turns sluggish). Recomputed automatically if the mass or
+           dimensions change. -->
+      <inertia ixx="${mass_base/12 * (base_width*base_width + base_height*base_height)}" ixy="0" ixz="0"
+               iyy="${mass_base/12 * (base_length*base_length + base_height*base_height)}" iyz="0"
+               izz="${mass_base/12 * (base_length*base_length + base_width*base_width)}"/>
     </inertial>
     <visual>

Commit message: URDF: lidar mounted with yaw pi -- the scan's +x points to the robot's back
Found in 2026-09-30's bags: on straight drives, ICP between consecutive
scans put the lidar's motion at -176 deg in its own frame (230/239
segments, three runs) while the wheels said forward. With yaw 0, SLAM's
heading drifted against the (correct) IMU/EKF heading by hundreds of
degrees -- the rotated/duplicated lanes and lost heading -- and Nav2 saw
obstacles ahead as behind. Turns looked right either way (a 180 deg
offset doesn't flip rotation), which is why scan-vs-gyro turn checks
passed. The sim lidar is 360 deg, so the sim is unaffected.

replay_mapping.sh: retry the slam_toolbox active check (activation can
lag the 'successful' reply on a busy machine).

Co-Authored-By: Claude Opus 5.5 <noreply@anthropic.com>

File: src/bot_gazebo/urdf/bot.urdf.xacro (robot description, xacro)
@@ -224,7 +224,14 @@
        so the beam clears the camera. Measured position: see the sensor
        placement properties at the top of this file. The live scan confirms
-       no self-returns (nothing closer than 0.32 m, 2026-09-25). -->
+       no self-returns (nothing closer than 0.32 m, 2026-09-25).
+       Yaw pi (2026-10-01): the scan's +x points to the robot's BACK. In
+       yesterday's bags, ICP between consecutive scans on straight drives
+       put the lidar's travel at -176 deg in its own frame (230 of 239
+       segments) while the wheels said forward; with yaw 0, SLAM fought the
+       IMU heading by hundreds of degrees (rotated, duplicated lanes) and
+       Nav2 saw obstacles ahead as behind. Turns looked right either way
+       (a 180 deg mount doesn't flip rotation), which hid it. -->
   <joint name="lidar_joint" type="fixed">
-    <origin xyz="${oak_front_x - 0.035} ${oak_width/2 - 0.055} ${lidar_top_height - lidar_plane_below_top}" rpy="0 0 0"/>
+    <origin xyz="${oak_front_x - 0.035} ${oak_width/2 - 0.055} ${lidar_top_height - lidar_plane_below_top}" rpy="0 0 ${pi}"/>
     <parent link="base_link"/>
     <child link="lidar_link"/>
